File: PCB/PCB.sch (KiCad schematic (older format))
At the start: 43 parts, among them J1 USB_C_Receptacle_USB2.0, J2 USB_A, J3 USB_A, SW1 SW_Push, U1 ATMEGA32U4, U2 CY7C65632-28LTXCT, U3 TPD2S017, Y1 16MHz, Y2 16MHz

Commit message: Clear .sch file
Parts:
- removed C1, C13, C14, C16, C7: 1u, Capacitor_SMD:C_0603_1608Metric, symbol Device:C
- removed C10, C11, C12, C15, C17, C2, C3: 100n, Capacitor_SMD:C_0603_1608Metric, symbol Device:C
- removed C18, C4: 10u, Capacitor_SMD:C_0603_1608Metric, symbol Device:C
- removed C5, C6, C8, C9: 22p, Capacitor_SMD:C_0603_1608Metric, symbol Device:C
- removed F1: 500mA, keyboard:Fuse_0805_2012Metric, symbol Device:Polyfuse_Small
- removed FB1, FB2, FB3: 600R, josh-passives-smt:Ferrite_Bead_0603, symbol josh-passive:Ferrite_Bead_PWR
- removed J1: USB_C_Receptacle_USB2.0, josh-connectors:USB_C_Receptacle_GT-USB-7010, symbol Connector:USB_C_Receptacle_USB2.0
- removed J2, J3: USB_A, symbol Connector:USB_A
- removed R1, R6, R7: 10K, Resistor_SMD:R_0603_1608Metric, symbol Device:R
- removed R10: 649R, Resistor_SMD:R_0603_1608Metric, symbol Device:R
- removed R11, R8, R9: 100K, Resistor_SMD:R_0603_1608Metric, symbol Device:R
- removed R2, R3: 22R, Resistor_SMD:R_0603_1608Metric, symbol Device:R
- removed R4, R5: 5K1, Resistor_SMD:R_0603_1608Metric, symbol Device:R
- removed RN1: 10K, Resistor_SMD:R_Array_Convex_4x0402, symbol Device:R_Pack04
- removed SW1: SW_Push, josh-buttons-switches:BT_Small_2_Pin, symbol Switch:SW_Push
- removed U1: ATMEGA32U4, Package_QFP:TQFP-44_10x10mm_P0.8mm, symbol keyboard:ATMEGA32U4
- removed U2: CY7C65632-28LTXCT, Package_DFN_QFN:QFN-28-1EP_5x5mm_P0.5mm_EP3.35x3.35mm_ThermalVias, symbol josh-ic:CY7C65632-28LTXCT
- removed U3: TPD2S017, Package_TO_SOT_SMD:SOT-23-6, symbol Power_Protection:TPD2S017
- removed Y1, Y2: 16MHz, symbol Device:Crystal_GND24_Small
Connections:
- net labels removed: +3.3V, +3.3VA, +5V, D1_D+, D1_D-, D2_D+, D2_D-, GANG, GND, MISO, MOSI, RST, SCK, UP_USB_N, UP_USB_P, USB_DN_D+, USB_DN_D-, USB_UP_D+, USB_UP_D-, VBUS, VREG_3V3, XIN, XOUT, nOVR_1, nOVR_2, nOVR_3, nOVR_4
- wire segments 246 -> 0
- no-connect marks 13 -> 0
Other:
- note removed: "(Not used / disabled)"
- note removed: "Additional Ports"
- note removed: "Figure out which\none to place"
- note removed: "From Main USB Port"
- note removed: "MCU\n"
- note removed: "Main USB\n"
- note removed: "Microcontroller\n"
- note removed: "Over Current Detection"
- note removed: "To MCU\n"
- note removed: "Type-C\n"
- note removed: "USB Hub"
- note removed: "USB Hub Power"
- note removed: "USB Hub\n"

Commit message: Append nRFMicro schematic
Parts:
- added C1, C3: 10uF, Capacitor_SMD:C_0603_1608Metric, symbol nrfmicro-rescue:C
- added C2: 10uF, Capacitor_SMD:C_0603_1608Metric, symbol Device:C
- added D1: 1N5819, Diode_SMD:D_SOD-123, symbol nrfmicro-rescue:MBR0520
- added D2: BT, LED_SMD:LED_0603_1608Metric, symbol Device:LED
- added D3: CHG, LED_SMD:LED_0603_1608Metric, symbol Device:LED
- added D? (x48): 1n4148, symbol Device:D_Small
- added J2: USB-C USB 2.0 MC-372, nrfmicro:HRO-TYPE-C-31-M-12, symbol nrfmicro:HRO-TYPE-C-31-M-12
- added J3: Conn_01x04, nrfmicro:connector_swd, symbol Connector_Generic:Conn_01x02
- added J4: Conn_01x02, nrfmicro:connector_bat, symbol Connector_Generic:Conn_01x02
- added Q1: AO3407, Package_TO_SOT_SMD:SOT-23, symbol nrfmicro-rescue:BSS83P
- added Q2: AO3406, Package_TO_SOT_SMD:SOT-23, symbol Transistor_FET:BS870
- added R1, R3: 100K, Resistor_SMD:R_0603_1608Metric, symbol nrfmicro-rescue:R
- added R2: 4.7K, Resistor_SMD:R_0603_1608Metric, symbol Device:R
- added R4, R5: 5.1K, Resistor_SMD:R_0603_1608Metric, symbol Device:R
- added R6, R7: 1K, Resistor_SMD:R_0603_1608Metric, symbol Device:R
- added R8: 10K, Resistor_SMD:R_0603_1608Metric, symbol nrfmicro-rescue:R
- added R9: 10K, Resistor_SMD:R_0603_1608Metric, symbol Device:R
- added SW1: MSK-12C02, nrfmicro:switch_MSK-12C02_smd, symbol Switch:SW_SPDT
- added SW? (x48): SW_Push, symbol Switch:SW_Push
- added U1: E73-2G4M08S1C, nrfmicro:E73-2G4M08S1C-52840, symbol nrfmicro:E73-2G4M08S1C-52840
- added U2: MCP73831, Package_TO_SOT_SMD:SOT-23-5, symbol Battery_Management:MCP73831-2-OT
- added U3: AP2112K-3.3, Package_TO_SOT_SMD:SOT-23-5, symbol Regulator_Linear:AP2112K-3.3
Connections:
- new net: C3.1, D1.1 (K), Q1.2 (S), R1.1, U3.1 (VIN)
- new net: Q1.3 (D), R8.1, SW1.3 (C)
- new net: R2.1, U2.5 (PROG)
- new net: R7.2, U2.1 (STAT)
- new net: J2.10 (CC2), R5.1
- new net: J2.4 (CC1), R4.1
- new net: D3.1 (K), R7.1
- new net: D2.1 (K), R6.1
- new net: R1.2, U3.3 (EN)
- new net: SW?.1, SW?.1, SW?.1 (x5)
- new net: D?.2 (A), SW?.2 (x48)
- new net: D?.1 (K), D?.1 (K), D?.1 (K), D?.1 (K), D?.1 (K), D?.1 (K), D?.1 (K), D?.1 (K), D?.1 (K), D?.1 (K), D?.1 (K), D?.1 (K), D?.1 (K), D?.1 (K)
- new net: SW?.1, SW?.1, SW?.1, SW?.1 (x8)
- new net: D?.1 (K), D?.1 (K), D?.1 (K), D?.1 (K), D?.1 (K), D?.1 (K), D?.1 (K), D?.1 (K), D?.1 (K), D?.1 (K), D?.1 (K), D?.1 (K), D?.1 (K) (x2)
- new net: D?.1 (K), D?.1 (K), D?.1 (K), D?.1 (K), D?.1 (K), D?.1 (K), D?.1 (K), D?.1 (K)
- new net BLUE_LED: D2.2 (A), U1.2 (P1.10)
- new net BOOT: U1.22 (P0.07)
- new net DATA+: J2.6 (DP1), J2.8 (DP2), U1.31 (USB_D+)
- new net DATA-: J2.5 (DN2), J2.7 (DN1), U1.29 (USB_D-)
- new net DFU: U1.38 (P1.02)
- new net EXT_GND: Q2.3 (D)
- new net GND: C1.2, C2.2, C3.2, J2.1 (GND), J2.12 (GND), J4.2 (Pin_2), Q2.2 (S), R2.2, R3.2, R4.2, R5.2, R6.2, U1.21 (GND), U1.24 (GND), U1.5 (GND), U2.2 (VSS), U3.2 (GND)
- new net P0.00: U1.11 (P0.00/XL1)
- new net P0.01: U1.13 (P0.01/XL2)
- new net P0.02: U1.7 (P0.02/AIN0)
- new net P0.03: U1.3 (P0.03/AIN1)
- new net P0.04: R8.2, U1.12 (P0.26), U1.18 (P0.04/AIN2)
- new net P0.05: U1.15 (P0.05/AIN3)
- new net P0.09: U1.41 (P0.09/NFC1)
- new net P0.10: U1.43 (P0.10/NFC2)
- new net P0.12: U1.20 (P0.12)
- new net P0.13: U1.33 (P0.13)
- new net P0.15: U1.28 (P0.15)
- new net P0.17: U1.30 (P0.17)
- new net P0.20: U1.32 (P0.20)
- new net P0.22: U1.34 (P0.22)
- new net P0.24: U1.35 (P0.24)
- new net P0.28: U1.4 (P0.28/AIN4)
- new net P0.29: U1.8 (P0.29/AIN5)
- new net P0.30: U1.10 (P0.30/AIN6)
- new net P0.31: U1.9 (P0.31/AIN7)
- new net P1.04: U1.40 (P1.04)
- new net P1.06: U1.42 (P1.06)
- new net P1.11: U1.1 (P1.11)
- new net P1.13: U1.6 (P1.13)
- new net POWER_PIN: Q2.1 (G), R9.2, U1.17 (P1.09)
- new net RESET: U1.26 (P0.18/RESET)
- new net RXD: U1.16 (P0.08)
- new net SWC: J3.1 (Pin_1), U1.39 (SWDCLK)
- new net SWD: J3.2 (Pin_2), U1.37 (SWDIO)
- new net SWO: U1.36 (P1.00)
- new net TXD: U1.14 (P0.06)
- new net VBAT: C2.1, J4.1 (Pin_1), SW1.2 (B), U2.3 (VBAT)
- new net VBUS: D1.2 (A), D3.2 (A), J2.11 (VBUS), J2.2 (VBUS), Q1.1 (G), R3.1, U1.27 (VBUS), U2.4 (VDD)
- new net VCC: C1.1, R9.1, U1.19 (VDD), U3.5 (VOUT)
- no-connect marks 0 -> 7
Other:
- note added: "LiPo Charging\n"
- note added: "Power Control\nNormally On\nLow - Off\n"
- note added: "Power and Filtering"
