File: PCB/PCB.kicad_pcb (KiCad board)
At the start: 2 copper layers, 266.7 x 81.4 mm, 124 parts, among them J1 USB-C USB 2.0 MC-372, J2 Conn_01x04, J3 Conn_01x02, Q1 AO3407, Q2 AO3406, SW1 SW_Push, SW10 SW_Push, SW11 SW_Push, SW12 SW_Push, SW13 SW_Push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

Commit message: Unfill all zones, increase angle radius
Parts:
- removed G***: LOGO, Infinity:InfinityText
Other:
- outline, holes or cut-outs redrawn
